File: rapid_tank_level_indicator_hardware/rapid_tank_level_indicator.kicad_pcb (KiCad board)
At the start: 2 copper layers, 56 x 617 mm, 83 parts, among them J1 Conn_01x04_Pin, J17 TC2050, J2 Conn_02x04_Top_Bottom, J3 Conn_02x04_Top_Bottom, SW1 KMR721NGLFS, SW2 KMR721NGLFS, U1 L7805, U10 MCP9700Ax-ETT, U11 TPD4E1U06, U12 MCP9700Ax-ETT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

Commit message: finish design
Parts:
- added H1: MountingHole_Pad, MountingHole:MountingHole_3.2mm_M3_Pad_Via, F.Cu at (157.0, 56.0)
- added H2: MountingHole_Pad, MountingHole:MountingHole_3.2mm_M3_Pad_Via, F.Cu at (157.0, 13.9)
- added H3: MountingHole_Pad, MountingHole:MountingHole_3.2mm_M3_Pad_Via, F.Cu at (114.9, 13.9)
- added H4: MountingHole_Pad, MountingHole:MountingHole_3.2mm_M3_Pad_Via, F.Cu at (114.8, 56.2)
- moved U14 115.2 mm to (134.4, 415.1)
- moved R5 70.8 mm to (133.4, 415.2), turned to -90 degrees
- moved D10 70.1 mm to (134.6, 415.2), turned to -90 degrees
- moved R6 61.4 mm to (133.4, 356.8), turned to -90 degrees
- moved D11 60.6 mm to (134.6, 356.8), turned to -90 degrees
- moved R26 54.3 mm to (133.2, 648.4), turned to -90 degrees
- moved D9 53.2 mm to (134.4, 648.4), turned to -90 degrees
- moved R7 52.3 mm to (133.6, 298.4), turned to -90 degrees
- moved D12 51.4 mm to (134.8, 298.4), turned to -90 degrees
- moved U7 48.7 mm to (134.4, 298.4)
- moved U4 48.6 mm to (134.4, 648.4)
- moved R9 46.7 mm to (133.6, 240.3), turned to -90 degrees
- moved D13 45.6 mm to (134.8, 240.3), turned to -90 degrees
- moved R30 42.5 mm to (133.4, 590.1), turned to -90 degrees
- moved D1 41.4 mm to (134.6, 590.1), turned to -90 degrees
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Connections:
- U11 pad 1: /J1-SWO -> /J1-SWDIO
- U11 pad 2: /J1-SWDIO -> /J1-SWO
- U16 pad 1: CAN1_TX -> CAN2_TX
- U16 pad 4: CAN1_RX -> CAN2_RX
- U3 pad 10: TEMP_3 -> STAT_LED7
- U3 pad 11: TEMP_4 -> STAT_LED8
- U3 pad 14: TEMP_5 -> STAT_LED9
- U3 pad 15: TEMP_6 -> STAT_LED10
- U3 pad 16: TEMP_7 -> unconnected-(U3-PA2-Pad16)
- U3 pad 17: TEMP_8 -> TEMP_9
- U3 pad 2: STAT_LED6 -> unconnected-(U3-PC13-Pad2)
- U3 pad 20: TEMP_9 -> TEMP_8
- U3 pad 21: TEMP_10 -> TEMP_7
- U3 pad 22: AIN1 -> TEMP_6
- U3 pad 23: AIN0 -> TEMP_5
- U3 pad 24: unconnected-(U3-PC4-Pad24) -> TEMP_4
- U3 pad 25: unconnected-(U3-PC5-Pad25) -> TEMP_3
- U3 pad 26: STAT_LED9 -> TEMP_2
- U3 pad 27: unconnected-(U3-PB1-Pad27) -> TEMP_1
- U3 pad 28: unconnected-(U3-PB2-Pad28) -> STAT_LED6
- U3 pad 29: unconnected-(U3-PB10-Pad29) -> STAT_LED5
- U3 pad 3: STAT_LED7 -> unconnected-(U3-PC14-Pad3)
- U3 pad 30: unconnected-(U3-PB11-Pad30) -> STAT_LED4
- U3 pad 33: unconnected-(U3-PB12-Pad33) -> STAT_LED3
- U3 pad 34: unconnected-(U3-PB13-Pad34) -> STAT_LED2
- U3 pad 35: unconnected-(U3-PB14-Pad35) -> STAT_LED1
- U3 pad 37: SWITCH -> unconnected-(U3-PC6-Pad37)
- U3 pad 38: STAT_LED10 -> unconnected-(U3-PC7-Pad38)
- U3 pad 39: STAT_LED1 -> unconnected-(U3-PC8-Pad39)
- U3 pad 4: STAT_LED8 -> unconnected-(U3-PC15-Pad4)
- U3 pad 40: STAT_LED2 -> unconnected-(U3-PC9-Pad40)
- U3 pad 41: ADC -> unconnected-(U3-PA8-Pad41)
- U3 pad 51: STAT_LED3 -> unconnected-(U3-PC10-Pad51)
- U3 pad 52: STAT_LED4 -> unconnected-(U3-PC11-Pad52)
- U3 pad 53: STAT_LED5 -> unconnected-(U3-PC12-Pad53)
- U3 pad 57: unconnected-(U3-PB5-Pad57) -> CAN2_RX
- U3 pad 58: unconnected-(U3-PB6-Pad58) -> CAN2_TX
- U3 pad 61: CAN1_RX -> unconnected-(U3-PB8-Pad61)
- U3 pad 62: CAN1_TX -> unconnected-(U3-PB9-Pad62)
- U3 pad 8: TEMP_1 -> TEMP_10
- U3 pad 9: TEMP_2 -> unconnected-(U3-PC1-Pad9)
Routing:
- net +3.3V: track 0.00 -> 790.9 mm, vias 0 -> 2
- net +5V: track 0.00 -> 766.4 mm, vias 0 -> 9
- net STAT_LED1: track 0.00 -> 610.6 mm, vias 0 -> 2
- net TEMP_1: track 0.00 -> 601.5 mm, vias 0 -> 1
- net STAT_LED2: track 0.00 -> 551.6 mm, vias 0 -> 2
- net TEMP_2: track 0.00 -> 543.0 mm, vias 0 -> 1
- net STAT_LED3: track 0.00 -> 492.1 mm, vias 0 -> 2
- net TEMP_3: track 0.00 -> 484.4 mm, vias 0 -> 1
- net STAT_LED4: track 0.00 -> 426.9 mm
- net TEMP_4: track 0.00 -> 426.0 mm, vias 0 -> 1
- net STAT_LED5: track 0.00 -> 368.2 mm
- net TEMP_5: track 0.00 -> 367.9 mm, vias 0 -> 1
- net STAT_LED6: track 0.00 -> 309.7 mm
- net TEMP_6: track 0.00 -> 309.6 mm, vias 0 -> 1
- net STAT_LED7: track 0.00 -> 258.2 mm
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- added copper zone on B.Cu, net GND
- added copper zone on F.Cu, net GND
Other:
- board size 56 x 617 mm -> 50 x 643 mm
- board text added: "Bend zone"
- board text added: "Bulk head zone"
- board text added: "Edge"
- board text added: "Measure range"
- board text removed: "BOOT"
- board text removed: "RST"
