File: rapid_tank_level_indicator_hardware/rapid_tank_level_indicator.kicad_pcb (KiCad board)
At the start: 2 copper layers, 50 x 643.1 mm, 97 parts, among them J1 Conn_01x04_Pin, J17 TC2050, J2 Conn_02x04_Top_Bottom, J3 Conn_02x04_Top_Bottom, J4 Conn_01x12, J5 FFC3B07-12-T, SW1 KMR721NGLFS, SW2 KMR721NGLFS, U1 L7805, U10 MCP9700Ax-ETT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

Commit message: check LCSC parts and small layout adjustments
Parts:
- removed C12, C2, C24, C25, C29, C3, C4, C5: 100n, Capacitor_SMD:C_0402_1005Metric
- removed R1: 1k5, Resistor_SMD:R_0402_1005Metric
- added C31: 10p, Capacitor_SMD:C_0402_1005Metric, F.Cu at (132.9, 47.9)
- added C32: 100n, Capacitor_SMD:C_0402_1005Metric, F.Cu at (140.3, 39.2)
- added C33: 100n, Capacitor_SMD:C_0402_1005Metric, F.Cu at (136.9, 42.1)
- added C34: 100n, Capacitor_SMD:C_0402_1005Metric, F.Cu at (147.9, 53.7)
- added C35: 100n, Capacitor_SMD:C_0402_1005Metric, F.Cu at (124.8, 42.9)
- added C36: 100n, Capacitor_SMD:C_0402_1005Metric, F.Cu at (149.9, 37.1)
- added C37: 100n, Capacitor_SMD:C_0402_1005Metric, F.Cu at (136.2, 30.6)
- added C38: 100n, Capacitor_SMD:C_0402_1005Metric, F.Cu at (129.4, 32.0)
- added G***: LOGO, frodo_io_module:rapid_logo, B.Cu at (142.8, 34.8)
- added R17: 10k, Resistor_SMD:R_0402_1005Metric, F.Cu at (136.6, 54.6)
- added TP_3V3: 3V3, TestPoint:TestPoint_Pad_D1.5mm, F.Cu at (117.8, 31.1)
- added TP_5V1: 5V, TestPoint:TestPoint_Pad_D1.5mm, F.Cu at (128.2, 41.5)
- added TP_CAN_H1: CAN_H, TestPoint:TestPoint_Pad_D1.5mm, F.Cu at (124.5, 29.6)
- added TP_CAN_L1: CAN_L, TestPoint:TestPoint_Pad_D1.5mm, F.Cu at (126.5, 31.7)
- C20: value 10p -> 100n
- R15: value 10k -> 1k
- moved R15 12.9 mm to (124.8, 49.3), turned to 90 degrees
- moved C20 9.82 mm to (140.9, 53.8)
- moved C9 6.51 mm to (134.7, 52.8)
- moved R40 0.80 mm to (132.6, 35.3)
Connections:
- C20 pad 1: Net-(C20-Pad1) -> +3.3V
- R15 pad 1: TEMP_10_con -> Net-(D3-A)
- R15 pad 2: Net-(U3-PC0) -> Net-(D2-A)
- R25 pad 2: Net-(C20-Pad1) -> Net-(C31-Pad1)
- Y1 pad 1: Net-(C20-Pad1) -> Net-(C31-Pad1)
Routing:
- net CAN_1+: track 34.9 -> 44.4 mm, vias 0 -> 2
- net CAN_1-: track 38.5 -> 43.1 mm
- net +3.3V: track 188.5 -> 193.0 mm
- net Net-(C31-Pad1): track 0.00 -> 3.77 mm
- net Net-(C20-Pad1): track 3.77 -> 0.00 mm
- net GND: track 71.0 -> 73.7 mm, vias 147 -> 311
- net +5V: track 133.0 -> 134.6 mm
- added copper zone on F.Cu, net +3.3V
Other:
- board text added: "3.3V"
- board text added: "3V3"
- board text added: "5V"
- board text added: "CAN_H"
- board text added: "CAN_L"
- board text added: "CLK"
- board text added: "DIO"
- board text added: "Rapid tank level indicator"
- board text added: "Ref 1"
- board text added: "S1"
- board text added: "S2"
- board text removed: "T1"
- board text removed: "T10"
- board text removed: "Top"
