File: rapid_tank_level_indicator_hardware/rapid_tank_level_indicator.kicad_sch (KiCad schematic)
At the start: 97 parts, among them J1 Conn_01x04_Pin, J17 TC2050, J2 Conn_02x04_Top_Bottom, J3 Conn_02x04_Top_Bottom, J4 Conn_01x12, J5 FFC3B07-12-T, SW1 KMR721NGLFS, SW2 KMR721NGLFS, U1 L7805, U10 MCP9700Ax-ETT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

Commit message: check LCSC parts and small layout adjustments
Parts:
- removed C12, C24, C25, C29: 100n, Capacitor_SMD:C_0402_1005Metric, symbol Device:C_Small
- removed C2, C3, C4, C5: 100n, Capacitor_SMD:C_0402_1005Metric, symbol Device:C
- removed R1: 1k5, Resistor_SMD:R_0402_1005Metric, symbol Device:R_Small
- removed R15: 10k, Resistor_SMD:R_0402_1005Metric, symbol Device:R
- added C31: 10p, Capacitor_SMD:C_0402_1005Metric, symbol Device:C
- added C32, C33, C34, C35, C36, C37, C38: 100n, Capacitor_SMD:C_0402_1005Metric, symbol Device:C
- added R15: 1k, Resistor_SMD:R_0402_1005Metric, symbol Device:R_Small
- added R17: 10k, Resistor_SMD:R_0402_1005Metric, symbol Device:R
- added TP_3V3: 3V3, TestPoint:TestPoint_Pad_D1.5mm, symbol Connector:TestPoint
- added TP_5V1: 5V, TestPoint:TestPoint_Pad_D1.5mm, symbol Connector:TestPoint
- added TP_CAN_H1: CAN_H, TestPoint:TestPoint_Pad_D1.5mm, symbol Connector:TestPoint
- added TP_CAN_L1: CAN_L, TestPoint:TestPoint_Pad_D1.5mm, symbol Connector:TestPoint
- C1: LCSC (none) -> C23733; LCSC# C368809 -> (none); Manufacturer Samsung Electro-Mechanics -> (none); basic? (none) -> Yes
- C10, C7: LCSC (none) -> C15195; LCSC# C60133 -> (none); Manufacturer YAGEO -> (none); basic (none) -> yes
- C11: LCSC (none) -> C159798; LCSC# C159798 -> (none); basic (none) -> no
- C13, C14, C18, C19, C22, C23, C26, C27, C28, C30: Basic? (none) -> yes; LCSC (none) -> C52923
- C15: Basic? (none) -> Yes
- C16: Basic? (none) -> Yes; LCSC C76991 -> C15525; Manufacturer Murata Electronics -> (none); Part# CL31B106KAHNNNE -> (none)
- C17: Basic? (none) -> No
- C20: value 10p -> 100n; LCSC (none) -> C307331; LCSC# C76946 -> (none); Manufacturer Murata Electronics -> (none); basic (none) -> yes
- C21: LCSC (none) -> C32949; LCSC# C76946 -> (none); Manufacturer Murata Electronics -> (none); basic (none) -> yes
- C6: LCSC (none) -> C307331; LCSC# C77020 -> (none); Manufacturer Murata Electronics -> (none); basic (none) -> yes
- C8, C9: LCSC (none) -> C52923; LCSC# C52923 -> (none); basic (none) -> yes
- D16: LCSC (none) -> C5140034; LCSC# C5140034 -> (none); basic (none) -> no
- D2: LCSC (none) -> C162059; LCSC # C162059 -> (none); basic (none) -> no
- D3: Basic? (none) -> yes; LCSC (none) -> C2286; LCSC# C2286 -> (none)
- D4, D5, R12, R3, R41, R46, R47: basic (none) -> yes
- F1: LCSC (none) -> C311062; LCSC# C311062 -> (none); basic (none) -> no
- FB1: LCSC (none) -> C14709; LCSC# C14709 -> (none); basic? (none) -> yes
- J1, J4: now not fitted
- J2, J3: LCSC# x -> (none); now not fitted
- J5: LCSC (none) -> C5641303; basic (none) -> no
- R10, R11: Basic (none) -> Yes; LCSC (none) -> C25744
- R13, R9: #LCSC C25744 -> (none); Basic (none) -> Yes; LCSC (none) -> C25744
- R14: #LCSC C25744 -> (none); Basic? (none) -> yes; LCSC (none) -> C25744
- R16: Basic? (none) -> Yes; LCSC (none) -> C25091; LCSC# C112291 -> (none); Manufacturer ROHM Semicon -> (none); Part# ESR03EZPJ221 -> (none)
- R2: basic? (none) -> yes
- R25: LCSC (none) -> C21190; LCSC# C21190 -> (none); basic (none) -> yes
- R4, R5, R7: #LCSC C25744 -> (none); LCSC (none) -> C25744
- R40: LCSC (none) -> x; LCSC# x -> (none)
- R6: #LCSC C25744 -> (none); LCSC (none) -> C25744; basic? (none) -> yes
- R8: basic (none) -> Yes
- SW2, U5: Basic (none) -> No
- U10, U11: basic (none) -> no
- U16: LCSC (none) -> C191417; LCSC# C191417 -> (none); basic (none) -> no
- U3: LCSC (none) -> C8345; LCSC# C8345 -> (none); basic (none) -> no
- Y1: LCSC (none) -> C2149245; LCSC# C2149245 -> (none); basic (none) -> no
Connections:
- net +3.3V: now also C20.1, C32.1, C33.1, C34.1, C38.1, TP_3V3.1
- net +5V: now also C36.1, C37.1, TP_5V1.1
- net CAN_1+: now also TP_CAN_H1.1
- net CAN_1-: now also TP_CAN_L1.1
- net GND: now also C31.2, C32.2, C33.2, C34.2, C35.2, C36.2, C37.2, C38.2
- net TEMP_10_con: now also R17.1
- net at C30.1, U3.8 (PC0): now also R17.2
- net at D2.2 (A), U1.3 (OUT): now also C35.1, R15.2
- net at D3.2 (A): now also R15.1
- net at R25.2, Y1.1: now also C31.1; no longer C20.1
Other:
- note added: "@TODO"
- note added: "The selected part has only a 20% accuracy"
- note added: "We are using a higher resistance here, as the LED has to be that bright"
