File: rapid_tank_level_indicator_hardware/board/rapid_tank_level_indicator_board.kicad_pcb (KiCad board)
At the start: 2 copper layers, 50 x 59.2 mm, 81 parts, among them J1 Conn_01x04_Pin, J17 TC2050, J2 Conn_02x04_Top_Bottom, J3 Conn_02x04_Top_Bottom, J5 FFC3B07-12-T, SW1 KMR721NGLFS, SW2 KMR721NGLFS, U1 L7805, U11 TPD4E1U06, U16 MCP2562-E-SN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

Commit message: last edits
Parts:
- removed D2: RB070MM-30TR, Diode_SMD:D_SOD-123F
- R16: value 220 -> 1k
- moved R15 0.07 mm to (111.5, 78.5)
Connections:
- C35 pad 1: Net-(D2-A) -> +5V
- R15 pad 2: Net-(D2-A) -> +5V
- U1 pad 3: Net-(D2-A) -> +5V
Routing:
- net +5V: track 134.6 -> 143.2 mm
- net Net-(D2-A): track 8.51 -> 0.00 mm
- net SWDIO: track 25.8 -> 24.5 mm
- net Net-(U3-PA7): track 6.63 -> 5.62 mm
- net GND: vias 311 -> 308
Other:
- board text added: "CAN1"
- board text added: "CAN2"
- board text added: "h"
- board text added: "l"
- board text added: "rev 1"
- board text added: "vch"
- board text added: "vm"
- board text removed: "CAN1_h"
- board text removed: "CAN1_l"
- board text removed: "CAN2_h"
- board text removed: "CAN2_l"
- board text removed: "Ref 1"
- board text removed: "Vcharg"
- board text removed: "Vmain"
