File: rapid_tank_level_indicator_hardware/board/rapid_tank_level_indicator_board.kicad_sch (KiCad schematic)
At the start: 80 parts, among them J1 Conn_01x04_Pin, J17 TC2050, J2 Conn_02x04_Top_Bottom, J3 Conn_02x04_Top_Bottom, J5 FFC3B07-12-T, SW1 KMR721NGLFS, SW2 KMR721NGLFS, U1 L7805, U11 TPD4E1U06, U16 MCP2562-E-SN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

Commit message: last edits
Parts:
- removed D2: RB070MM-30TR, Diode_SMD:D_SOD-123F, symbol Diode:SS34
- H1, H2, H3, H4, J17, J5, SW1, SW2: now not fitted
- R16: value 220 -> 1k; LCSC C25091 -> C11702
- R25: LCSC C21190 -> C11702
Connections:
- net +5V: now also C35.1, R15.2, U1.3 (OUT)
Changed lines of the file:
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@@
 	)
 	(junction
+		(at 213.36 33.02)
+		(diameter 0)
+		(color 0 0 0 0)
+	)
+	(junction
 		(at 322.58 38.1)
 		(diameter 0)
@@
 	)
 	(junction
-		(at 205.74 33.02)
-		(diameter 0)
-		(color 0 0 0 0)
-	)
-	(junction
 		(at 209.55 121.92)
 		(diameter 0)
@@
 	(wire
 		(pts
-			(xy 205.74 33.02) (xy 207.01 33.02)
-		)
-		(stroke
-			(width 0)
-			(type default)
-		)
-	)
-	(wire
-		(pts
 			(xy 298.45 53.34) (xy 304.8 53.34)
 		)
@@
 	(wire
 		(pts
-			(xy 213.36 35.56) (xy 213.36 38.1)
-		)
-		(stroke
-			(width 0)
-			(type default)
-		)
-	)
-	(wire
-		(pts
 			(xy 237.49 163.83) (xy 250.19 163.83)
 		)
@@
 	(wire
 		(pts
-			(xy 214.63 33.02) (xy 218.44 33.02)
-		)
-		(stroke
-			(width 0)
-			(type default)
-		)
-	)
-	(wire
-		(pts
 			(xy 368.3 27.94) (xy 368.3 29.21)
 		)
@@
 	(wire
 		(pts
-			(xy 205.74 33.02) (xy 205.74 35.56)
+			(xy 213.36 33.02) (xy 213.36 38.1)
 		)
 		(stroke
@@
 	(wire
 		(pts
+			(xy 213.36 33.02) (xy 218.44 33.02)
+		)
+		(stroke
+			(width 0)
+			(type default)
+		)
+	)
+	(wire
+		(pts
 			(xy 373.38 88.9) (xy 381 88.9)
 		)
@@
 	(wire
 		(pts
-			(xy 201.93 33.02) (xy 205.74 33.02)
+			(xy 201.93 33.02) (xy 213.36 33.02)
 		)
 		(stroke
@@
 	(wire
 		(pts
-			(xy 205.74 35.56) (xy 213.36 35.56)
-		)
-		(stroke
-			(width 0)
-			(type default)
-		)
-	)
-	(wire
-		(pts
 			(xy 361.95 88.9) (xy 361.95 95.25)
 		)
@@
 			)
 		)
-		(property "Value" "220"
+		(property "Value" "1k"
 			(at 222.885 132.08 0)
 			(show_name no)
@@
 			)
 		)
-		(property "LCSC" "C25091"
+		(property "LCSC" "C11702"
 			(at 227.838 130.556 0)
 			(show_name no)
@@
 		(on_board yes)
 		(in_pos_files yes)
-		(dnp no)
+		(dnp yes)
 		(property "Reference" "H2"
 			(at 163.195 95.885 90)
@@
 		(on_board yes)
 		(in_pos_files yes)
-		(dnp no)
+		(dnp yes)
 		(property "Reference" "H3"
 			(at 163.195 100.965 90)
@@
 		(on_board yes)
 		(in_pos_files yes)
-		(dnp no)
+		(dnp yes)
 		(fields_autoplaced yes)
 		(property "Reference" "J17"
@@
 		(on_board yes)
 		(in_pos_files yes)
-		(dnp no)
+		(dnp yes)
 		(property "Reference" "J5"
 			(at 242.57 182.88 0)
@@
 		(on_board yes)
 		(in_pos_files yes)
-		(dnp no)
+		(dnp yes)
 		(property "Reference" "H1"
 			(at 163.195 90.805 90)
@@
 	)
 	(symbol
-		(lib_id "Diode:SS34")
-		(at 210.82 33.02 180)
-		(unit 1)
-		(body_style 1)
-		(exclude_from_sim no)
-		(in_bom yes)
-		(on_board yes)
-		(in_pos_files yes)
-		(dnp no)
-		(property "Reference" "D2"
-			(at 210.82 30.226 0)
-			(show_name no)
-			(do_not_autoplace no)
-			(effects
-				(font
-					(size 1.27 1.27)
-				)
-			)
-		)
-		(property "Value" "RB070MM-30TR"
-			(at 211.074 30.48 0)
-			(hide yes)
-			(show_name no)
-			(do_not_autoplace no)
-			(effects
-				(font
-					(size 1.27 1.27)
-				)
-			)
-		)
-		(property "Footprint" "Diode_SMD:D_SOD-123F"
-			(at 210.82 28.575 0)
-			(hide yes)
-			(show_name no)
-			(do_not_autoplace no)
-			(effects
-				(font
-					(size 1.27 1.27)
-				)
-			)
-		)
-		(property "Datasheet" "https://www.lcsc.com/datasheet/lcsc_datasheet_1809051324_ROHM-Semicon-RB070MM-30TR_C162059.pdf"
-			(at 210.82 33.02 0)
-			(hide yes)
-			(show_name no)
-			(do_not_autoplace no)
-			(effects
-				(font
-					(size 1.27 1.27)
-				)
-			)
-		)
-		(property "Description" "30V 490mV@1.5A 1.5A SOD-123F Schottky Diodes ROHS"
-			(at 210.82 33.02 0)
-			(hide yes)
-			(show_name no)
-			(do_not_autoplace no)
-			(effects
-				(font
-					(size 1.27 1.27)
-				)
-			)
-		)
-		(property "LCSC" "C162059"
-			(at 210.312 28.448 0)
-			(show_name no)
-			(do_not_autoplace no)
-			(effects
-				(font
-					(size 1.27 1.27)
-				)
-			)
-		)
-		(property "basic" "no"
-			(at 213.36 29.718 0)
-			(show_name no)
-			(do_not_autoplace no)
-			(effects
-				(font
-					(size 1.27 1.27)
-				)
-			)
-		)
-		(pin "1"
-		)
-		(pin "2"
-		)
-		(instances
-			(project "rapid_tank_level_indicator_board"
-				(path "/1c1f559e-6fe1-4cfb-8cad-aaff8e3c1892"
-					(reference "D2")
-					(unit 1)
-				)
-			)
-		)
-	)
-	(symbol
 		(lib_id "power:PWR_FLAG")
 		(at 184.15 41.91 180)
@@
 		(on_board yes)
 		(in_pos_files yes)
-		(dnp no)
+		(dnp yes)
 		(property "Reference" "SW2"
 			(at 250.063 99.4953 90)
@@
 		(on_board yes)
 		(in_pos_files yes)
-		(dnp no)
+		(dnp yes)
 		(property "Reference" "H4"
 			(at 163.195 106.045 90)
@@
 			)
 		)
-		(property "LCSC" "C21190"
+		(property "LCSC" "C11702"
 			(at 232.918 144.78 0)
 			(show_name no)
@@
 		(on_board yes)
 		(in_pos_files yes)
-		(dnp no)
+		(dnp yes)
 		(property "Reference" "SW1"
 			(at 243.713 63.9353 90)
