File: rapid_tank_level_indicator_hardware/sensor/rapid_tank_level_indicator_sensor.kicad_pcb (KiCad board)
At the start: 2 copper layers, 13 x 583.2 mm, 21 parts, among them J4 Conn_01x12, U10 MCP9700Ax-ETT, U12 MCP9700Ax-ETT, U13 MCP9700Ax-ETT, U14 MCP9700Ax-ETT, U15 MCP9700Ax-ETT, U4 MCP9700Ax-ETT, U6 MCP9700Ax-ETT, U7 MCP9700Ax-ETT, U8 MCP9700Ax-ETT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

Commit message: last edits
Routing:
- net +5V_post_con: track 619.4 -> 620.6 mm
- net GND_pos_con: vias 96 -> 115
Other:
- board text added: "Stiffener: Polyimide"
Changed lines of the file:
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@@
 		(filling no)
 		(pcbplotparams
-			(layerselection 0x00000000_00000000_55555555_5755f5ff)
+			(layerselection 0x00000000_00000000_55575555_5755f5ff)
 			(plot_on_all_layers_selection 0x00000000_00000000_00000000_00000000)
 			(disableapertmacros no)
@@
 			(plotpadnumbers no)
 			(hidednponfab no)
-			(sketchdnponfab yes)
-			(crossoutdnponfab yes)
+			(sketchdnponfab no)
+			(crossoutdnponfab no)
 			(subtractmaskfromsilk no)
 			(outputformat 1)
 			(mirror no)
-			(drillshape 1)
+			(drillshape 0)
 			(scaleselection 1)
 			(outputdirectory "")
@@
 		)
 	)
-	(gr_text "Stiffener: Polyimide\nThickness: 0.20mm"
+	(gr_text "Stiffener: Polyimide"
 		(at 142.9 75.7 0)
 		(layer "User.6")
@@
 	)
 	(segment
+		(start 130.6 71.62)
+		(end 130.6 117.6875)
+		(width 0.5)
+		(layer "B.Cu")
+		(net "+5V_post_con")
+	)
+	(segment
 		(start 134.575 472.475)
 		(end 131.9 469.8)
@@
 	)
 	(segment
+		(start 130.5 71.52)
+		(end 130.6 71.62)
+		(width 0.5)
+		(layer "B.Cu")
+		(net "+5V_post_con")
+	)
+	(segment
 		(start 131.9 178.3)
 		(end 131.9 177.326497)
@@
 	)
 	(segment
-		(start 130.34809 117.43559)
-		(end 131.9 118.9875)
-		(width 0.5)
-		(layer "B.Cu")
-		(net "+5V_post_con")
-	)
-	(segment
 		(start 134.575 297.475)
 		(end 131.9 294.8)
@@
 	)
 	(segment
-		(start 130.34809 72.8)
-		(end 130.34809 117.43559)
+		(start 130.6 117.6875)
+		(end 131.9 118.9875)
 		(width 0.5)
 		(layer "B.Cu")
@@
 	)
 	(via
+		(at 132.9 588.8)
+		(size 0.6)
+		(drill 0.3)
+		(layers "F.Cu" "B.Cu")
+		(free yes)
+		(net "GND_pos_con")
+	)
+	(via
 		(at 130.7 648)
 		(size 0.6)
@@
 	)
 	(via
+		(at 132.9 530.5)
+		(size 0.6)
+		(drill 0.3)
+		(layers "F.Cu" "B.Cu")
+		(free yes)
+		(net "GND_pos_con")
+	)
+	(via
 		(at 136.9 476.9)
 		(size 0.6)
@@
 	)
 	(via
+		(at 135.2 298.4)
+		(size 0.6)
+		(drill 0.3)
+		(layers "F.Cu" "B.Cu")
+		(free yes)
+		(net "GND_pos_con")
+	)
+	(via
 		(at 141 418.7)
 		(size 0.6)
@@
 	)
 	(via
+		(at 135.2 123.4)
+		(size 0.6)
+		(drill 0.3)
+		(layers "F.Cu" "B.Cu")
+		(free yes)
+		(net "GND_pos_con")
+	)
+	(via
+		(at 135.2 473.4)
+		(size 0.6)
+		(drill 0.3)
+		(layers "F.Cu" "B.Cu")
+		(free yes)
+		(net "GND_pos_con")
+	)
+	(via
+		(at 135.3 531.7)
+		(size 0.6)
+		(drill 0.3)
+		(layers "F.Cu" "B.Cu")
+		(free yes)
+		(net "GND_pos_con")
+	)
+	(via
 		(at 132 116.4)
 		(size 0.6)
@@
 	)
 	(via
+		(at 133 121.7)
+		(size 0.6)
+		(drill 0.3)
+		(layers "F.Cu" "B.Cu")
+		(free yes)
+		(net "GND_pos_con")
+	)
+	(via
 		(at 130.6 236.2)
 		(size 0.6)
@@
 	)
 	(via
+		(at 135.2 415.1)
+		(size 0.6)
+		(drill 0.3)
+		(layers "F.Cu" "B.Cu")
+		(free yes)
+		(net "GND_pos_con")
+	)
+	(via
 		(at 130.5 351.7)
 		(size 0.6)
@@
 	)
 	(via
+		(at 132.9 472.1)
+		(size 0.6)
+		(drill 0.3)
+		(layers "F.Cu" "B.Cu")
+		(free yes)
+		(net "GND_pos_con")
+	)
+	(via
 		(at 135.5 177.5)
 		(size 0.6)
@@
 	)
 	(via
+		(at 132.9 297.1)
+		(size 0.6)
+		(drill 0.3)
+		(layers "F.Cu" "B.Cu")
+		(free yes)
+		(net "GND_pos_con")
+	)
+	(via
 		(at 135 107.2)
 		(size 0.6)
@@
 	)
 	(via
+		(at 135.2 240.1)
+		(size 0.6)
+		(drill 0.3)
+		(layers "F.Cu" "B.Cu")
+		(free yes)
+		(net "GND_pos_con")
+	)
+	(via
 		(at 136.5 410.4)
 		(size 0.6)
@@
 	)
 	(via
+		(at 135.3 590.1)
+		(size 0.6)
+		(drill 0.3)
+		(layers "F.Cu" "B.Cu")
+		(free yes)
+		(net "GND_pos_con")
+	)
+	(via
 		(at 141 468.7)
 		(size 0.6)
@@
 	)
 	(via
+		(at 132.8 355.5)
+		(size 0.6)
+		(drill 0.3)
+		(layers "F.Cu" "B.Cu")
+		(free yes)
+		(net "GND_pos_con")
+	)
+	(via
 		(at 130.5 177.7)
 		(size 0.6)
@@
 	)
 	(via
+		(at 132.8 180.5)
+		(size 0.6)
+		(drill 0.3)
+		(layers "F.Cu" "B.Cu")
+		(free yes)
+		(net "GND_pos_con")
+	)
+	(via
 		(at 141.2 236.4)
 		(size 0.6)
@@
 	)
 	(via
+		(at 135.2 648.4)
+		(size 0.6)
+		(drill 0.3)
+		(layers "F.Cu" "B.Cu")
+		(free yes)
+		(net "GND_pos_con")
+	)
+	(via
 		(at 132.1 651)
 		(size 0.6)
@@
 	)
 	(via
+		(at 132.8 238.8)
+		(size 0.6)
+		(drill 0.3)
+		(layers "F.Cu" "B.Cu")
+		(free yes)
+		(net "GND_pos_con")
+	)
+	(via
 		(at 135 651.6)
 		(size 0.6)
@@
 	)
 	(via
+		(at 135.2 181.8)
+		(size 0.6)
+		(drill 0.3)
+		(layers "F.Cu" "B.Cu")
+		(free yes)
+		(net "GND_pos_con")
+	)
+	(via
 		(at 140.5 126.7)
 		(size 0.6)
@@
 	)
 	(via
+		(at 132.9 413.9)
+		(size 0.6)
+		(drill 0.3)
+		(layers "F.Cu" "B.Cu")
+		(free yes)
+		(net "GND_pos_con")
+	)
+	(via
 		(at 136.9 301.8)
 		(size 0.6)
@@
 		(size 0.6)
 		(drill 0.3)
+		(layers "F.Cu" "B.Cu")
+		(free yes)
+		(net "GND_pos_con")
+	)
+	(via
+		(at 135.2 356.8)
+		(size 0.6)
+		(drill 0.3)
